File: board/ignis.sch (KiCad schematic (older format))
At the start: 21 parts, among them P1 GND, P2 HOT, P3 NEUTRAL, P4 LOAD, P5 SAFETY, U1 PIC18F13K22, U2 PS2815-1, U3 FODM3022, U4 TRIAC

Commit message: Layout done for Rev. 0 bench test board.
Parts:
- removed D?: ZENER, symbol ZENER
- removed P4: LOAD, symbol CONN_01X02
- removed P5: SAFETY, symbol CONN_01X02
- added C2, C3: 0.1 uF, Capacitors_SMD:C_0603, symbol C
- added C4, C5: 10 uF, Capacitors_SMD:C_0603, symbol C_Small
- added C6, C7: 100 nF, Capacitors_SMD:C_0603, symbol C_Small
- added LOAD1, LOAD2: LOAD, ugw:62409-1, symbol CONN_01X01
- added P11: POWER, Terminal_Blocks:TerminalBlock_Pheonix_MPT-2.54mm_4pol, symbol CONN_01X04
- added P7: TYPE K, ugw:PCC-SMP-TN, symbol CONN_01X02
- added Q1, Q2, Q3: BSS138, TO_SOT_Packages_SMD:SOT-23, symbol BSS138
- added R10, R11, R12, R7, R8, R9: 10K, Resistors_SMD:R_0603, symbol R_Small
- added SAFE1, SAFE2: SAFETY, ugw:62409-1, symbol CONN_01X01
- added U5, U6: MAX31855KASA, Power_Integrations:SO-8, symbol MAX31855KASA-RESCUE-ignis
- added U7: LD1117S50CTR, TO_SOT_Packages_SMD:SOT-223, symbol LD1117S50CTR
- added U8: LD1117S33CTR, TO_SOT_Packages_SMD:SOT-223, symbol LD1117S33CTR
- C1: footprint (none) -> Capacitors_SMD:C_0603
- P1, P2, P3: footprint (none) -> ugw:62409-1
- P10: renamed from P?; footprint (none) -> Pin_Headers:Pin_Header_Straight_1x06
- P6: renamed from P?; value TYPE R -> TYPE K; footprint (none) -> ugw:PCC-SMP-TN
- P8: renamed from P?; footprint (none) -> Terminal_Blocks:TerminalBlock_Pheonix_MPT-2.54mm_2pol
- P9: renamed from P?; footprint (none) -> Connect:PINHEAD1-6
- R1, R2, R3, R4: footprint (none) -> Resistors_SMD:R_0603
- R5, R6: renamed from R?; footprint (none) -> Resistors_SMD:R_0603
- U1: footprint (none) -> SMD_Packages:SSOP-20
- U3: footprint MFP4L -> ugw:FODM30XX
- U4: footprint (none) -> TO_SOT_Packages_THT:TO-220_Neutral123_Horizontal_LargePads
Connections:
- net +5V: now also C4.1, C7.1, P11.3 (P3), R7.2, R8.2, R9.2, U7.2 (VO), U8.3 (VI)
- net GND: now also C2.2, C3.2, C4.2, C5.2, C6.2, C7.2, P11.1 (P1), U5.1 (GND), U6.1 (GND), U7.1 (GND), U8.1 (GND); no longer P6.2 (P2)
- net at R3.1, U4.2: now also LOAD1.1 (P1)
- net at U3.2: now also Q3.1 (G), Q3.2 (S), R12.1; no longer U1.11 (RB6/SCK)
- net at P6.1 (P1): now also U5.3 (T+); no longer U1.13 (RB4/AN10/SDI)
- net at U1.2 (RA5/OSC1/CLKIN): now also Q1.3 (D), R9.1
- net at U1.3 (RA4/AN3/OSC2/CLKOUT): now also Q2.3 (D), R8.1
- net at U1.9 (RC7/AN9/SDO): now also Q3.3 (D), R7.1
- net at P2.1 (P1), R2.2: now also SAFE2.1 (P1)
- new net: P6.2 (P2), U5.2 (T-)
- new net: U1.11 (RB6/SCK), U5.5 (SCK), U6.5 (SCK)
- new net: U1.13 (RB4/AN10/SDI), U5.7 (SO), U6.7 (SO)
- new net: Q2.1 (G), Q2.2 (S), R11.1, U5.6 (~CS~)
- new net: P7.1 (P1), U6.3 (T+)
- new net: P7.2 (P2), U6.2 (T-)
- new net: Q1.1 (G), Q1.2 (S), R10.1, U6.6 (~CS~)
- new net: LOAD2.1 (P1), SAFE1.1 (P1)
- new net +12V: C6.1, P11.4 (P4), U7.3 (VI)
- new net +3V3: C2.1, C3.1, C5.1, P11.2 (P2), R10.2, R11.2, R12.2, U5.4 (VCC), U6.4 (VCC), U8.2 (VO)
- no-connect marks 0 -> 5
Other:
- note added: "FTDI\nInterface"
- note added: "Level Translator"
- note added: "Load Switch Circuit"
- note added: "Power Regulators"
- note added: "Programming Port"
- note added: "Thermocouple Interface Circuit"
- note added: "Zero-Cross Detection Circuit"
- note removed: "Load circuit using a random phase \nTRIAC output optocoupler\nto hi trip a TRIAC. No on board\nover-current protection other than \nan inline safety port."
- note removed: "Need a Non-isolating Zener supply to get +5V from mains if FTDI can't support the MCU."
- note removed: "This is the zero cross detection \ncircuit. It will spike low when \nthe AC crosses zero."
- moved on the sheet: P6, R3, R4, U3, U4
