File: board/ignis.kicad_pcb (KiCad board)
At the start: 2 copper layers, 43 parts, among them P1 GND, P10 PROG, P11 POWER, P2 HOT, P3 NEUTRAL, P6 TYPE K, P7 TYPE K, P8 DOOR, P9 FTDI, Q1 BSS138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

Commit message: Edge fix and plot for prototype.
Other:
- board outline added: 68 x 66 mm
Changed lines of the file:
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@@
     (links 96)
     (no_connects 1)
-    (area 0 0 0 0)
+    (area 117 62 197.25 134.9)
     (thickness 1.6)
-    (drawings 2)
+    (drawings 6)
     (tracks 341)
     (zones 0)
@@
     (visible_elements 7FFFFFFF)
     (pcbplotparams
-      (layerselection 0x00030_80000001)
+      (layerselection 0x010f0_80000001)
       (usegerberextensions false)
       (excludeedgelayer true)
@@
       (outputformat 1)
       (mirror false)
-      (drillshape 1)
+      (drillshape 0)
       (scaleselection 1)
-      (outputdirectory ""))
+      (outputdirectory plot/))
   )
   (net 0 "")
@@
     )
   )
+  (gr_line (start 117 128) (end 117 62) (angle 90) (layer Edge.Cuts) (width 0.15))
+  (gr_line (start 185 128) (end 117 128) (angle 90) (layer Edge.Cuts) (width 0.15))
+  (gr_line (start 185 62) (end 185 128) (angle 90) (layer Edge.Cuts) (width 0.15))
+  (gr_line (start 117 62) (end 185 62) (angle 90) (layer Edge.Cuts) (width 0.15))
   (dimension 68 (width 0.3) (layer Cmts.User)
     (gr_text "68.000 mm" (at 151 133.549999) (layer Cmts.User)
